Commit message: Update.

File: robolab/data/robots/mini3/urdf/mini3.urdf (robot description, URDF)
Before this commit: robot mini3_27, 24 links, 23 joints
Joints:
- joint left_ankle_pitch_joint: limit lower=-0.5236 upper=0.5236 effort=7 velocity=25.133 -> lower=-0.5236 upper=0.5236 effort=25 velocity=25.133
- joint left_ankle_roll_joint: limit lower=-0.2618 upper=0.2618 effort=7 velocity=25.133 -> lower=-0.2618 upper=0.2618 effort=25 velocity=25.133
- joint right_ankle_pitch_joint: limit lower=-0.5236 upper=0.5236 effort=7 velocity=25.133 -> lower=-0.5236 upper=0.5236 effort=25 velocity=25.133
- joint right_ankle_roll_joint: limit lower=-0.2618 upper=0.2618 effort=7 velocity=25.133 -> lower=-0.2618 upper=0.2618 effort=25 velocity=25.133

Commit message: Remove hip-roll collision.

File: robolab/data/robots/mini3/urdf/mini3.urdf (robot description, URDF)
Before this commit: robot mini3_27, 24 links, 23 joints
Links:
- link left_hip_roll_link: geometry visual mesh filename=../meshes/left_hip_roll_link.STL
- link right_hip_roll_link: geometry visual mesh filename=../meshes/right_hip_roll_link.STL
